File: USB_HUB.kicad_sch (KiCad schematic)
At the start: 13 parts, among them U5 FE1.1s, Y1 12MHz

Commit message: Schematic progress
I keep forgetting that I'm just making a panadapter here and not a full blown SDR...oops
Parts:
- removed Y1: 12MHz, symbol Device:Crystal_GND24
- added R44: 1M, libraries:Worthington_R_0402, symbol Device:R_Small_US
- R13, R14, R15, R16, R17: footprint (none) -> libraries:Worthington_R_0402
Connections:
- net 5V0 renamed +5V0
- net XIN renamed 12MHz_CLK_IN
- net 12MHz_CLK_IN: now also R44.2
- net XOUT: no longer names the net of U5.2 (XOUT)
- net XOUT: now also R44.1
