File: Z10000.kicad_sch (KiCad schematic)
At the start: 6 parts, among them U10 AD8007AKS-R2

Commit message: Schematic progress
Parts:
- U10: DigiKey (none) -> AD8007AKSZ-REEL7CT-ND
Connections:
- net at C46.2: now also R46.1
- net at U10.3 (+): now also R46.2
Other:
- moved on the sheet: C46, R46
Changed lines of the file:
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@@
 	(generator_version "10.0")
 	(paper "B")
+	(wire
+		(pts
+			(xy 233.68 83.82) (xy 246.38 83.82)
+		)
+		(stroke
+			(width 0)
+			(type default)
+		)
+	)
+	(wire
+		(pts
+			(xy 213.36 83.82) (xy 228.6 83.82)
+		)
+		(stroke
+			(width 0)
+			(type default)
+		)
+	)
 	(image
 		(at 87.63 209.55)
@@
 	(symbol
 		(lib_id "Device:C_Small")
-		(at 264.16 114.3 90)
+		(at 210.82 83.82 90)
 		(mirror x)
 		(unit 1)
@@
 		(dnp no)
 		(property "Reference" "C46"
-			(at 263.652 111.506 90)
+			(at 210.312 81.026 90)
 			(show_name no)
 			(do_not_autoplace no)
@@
 		)
 		(property "Value" "100n"
-			(at 264.668 111.506 90)
+			(at 211.328 81.026 90)
 			(show_name no)
 			(do_not_autoplace no)
@@
 		)
 		(property "Footprint" "libraries:Worthington_C_0402"
-			(at 264.16 114.3 0)
+			(at 210.82 83.82 0)
 			(hide yes)
 			(show_name no)
@@
 		)
 		(property "Datasheet" ""
-			(at 264.16 114.3 0)
+			(at 210.82 83.82 0)
 			(hide yes)
 			(show_name no)
@@
 		)
 		(property "Description" "Unpolarized capacitor, small symbol"
-			(at 264.16 114.3 0)
+			(at 210.82 83.82 0)
 			(hide yes)
 			(show_name no)
@@
 					(unit 1)
 				)
+				(path "/9dbbaad8-804a-4efe-a989-bc17c5acbd91/cbfc5903-0c0d-474c-b17e-16443ef993f6"
+					(reference "C69")
+					(unit 1)
+				)
 			)
 		)
@@
 					(unit 1)
 				)
+				(path "/9dbbaad8-804a-4efe-a989-bc17c5acbd91/cbfc5903-0c0d-474c-b17e-16443ef993f6"
+					(reference "C85")
+					(unit 1)
+				)
 			)
 		)
@@
 					(unit 1)
 				)
+				(path "/9dbbaad8-804a-4efe-a989-bc17c5acbd91/cbfc5903-0c0d-474c-b17e-16443ef993f6"
+					(reference "R50")
+					(unit 1)
+				)
 			)
 		)
@@
 			)
 		)
-		(property "Datasheet" "https://www.analog.com/media/en/technical-documentation/data-sheets/ad8007_8008.pdf"
+		(property "Datasheet" "https://www.analog.com/media/en/technical-documentation/data-sheets/AD8007_8008.pdf"
 			(at 257.81 82.55 0)
 			(hide yes)
@@
 			)
 		)
+		(property "DigiKey" "AD8007AKSZ-REEL7CT-ND"
+			(at 254 86.36 0)
+			(hide yes)
+			(show_name no)
+			(do_not_autoplace no)
+			(effects
+				(font
+					(size 1.27 1.27)
+				)
+			)
+		)
 		(pin "2"
 		)
@@
 					(unit 1)
 				)
+				(path "/9dbbaad8-804a-4efe-a989-bc17c5acbd91/cbfc5903-0c0d-474c-b17e-16443ef993f6"
+					(reference "U12")
+					(unit 1)
+				)
 			)
 		)
@@
 					(unit 1)
 				)
+				(path "/9dbbaad8-804a-4efe-a989-bc17c5acbd91/cbfc5903-0c0d-474c-b17e-16443ef993f6"
+					(reference "L16")
+					(unit 1)
+				)
 			)
 		)
@@
 	(symbol
 		(lib_id "Device:R_Small_US")
-		(at 254 114.3 90)
+		(at 231.14 83.82 90)
 		(unit 1)
 		(body_style 1)
@@
 		(dnp no)
 		(property "Reference" "R46"
-			(at 253.492 111.76 90)
+			(at 230.632 81.28 90)
 			(show_name no)
 			(do_not_autoplace no)
@@
 		)
 		(property "Value" "100"
-			(at 254.508 111.76 90)
+			(at 231.648 81.28 90)
 			(show_name no)
 			(do_not_autoplace no)
@@
 		)
 		(property "Footprint" "libraries:Worthington_R_0402"
-			(at 254 114.3 0)
+			(at 231.14 83.82 0)
 			(hide yes)
 			(show_name no)
@@
 		)
 		(property "Datasheet" ""
-			(at 254 114.3 0)
+			(at 231.14 83.82 0)
 			(hide yes)
 			(show_name no)
@@
 		)
 		(property "Description" "Resistor, small US symbol"
-			(at 254 114.3 0)
+			(at 231.14 83.82 0)
 			(hide yes)
 			(show_name no)
@@
 					(unit 1)
 				)
+				(path "/9dbbaad8-804a-4efe-a989-bc17c5acbd91/cbfc5903-0c0d-474c-b17e-16443ef993f6"
+					(reference "R49")
+					(unit 1)
+				)
