File: PiZero_RTL_Panadapter.kicad_pcb (KiCad board)
At the start: 2 copper layers, 65 x 30 mm, 173 parts, among them J1 JST GH 8 Position, J2 U.FL, J3 U.FL, Q1 S8050, U1 Raspberry Pi Zero 2W, U10 AD8007AKS-R2, U11 Converter_DCDC_RECOM_RPMx.x-x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, U11 RPM5.0-2.0, U2 AP2114H-3.3, U3 RTL2832U, U4 M24C02-WMN, U5 FE1.1s, U6 RTL8152B, U7 R820T2, U8 Si5351A, U9 TPS22929D, Y1 12MHz, Y2 25M, Y3 25MHz

Commit message: Schematic progress
Parts:
- moved REF** 13.4 mm to (124.6, 93.8)
- moved U11 3.15 mm to (125.0, 102.5)
Changed lines of the file:
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@@
 	(footprint "Converter_DCDC:Converter_DCDC_RECOM_RPMx.x-x.0"
 		(layer "F.Cu")
-		(at 125 99.35)
+		(at 125 102.5)
 		(descr "https://www.recom-power.com/pdf/Innoline/RPM-6.0.pdf")
 		(tags "dc-dc recom buck lga-25 pitch 2.29mm")
@@
 	(footprint "libraries:CAPMP7.6X4.3_4.3N_KEM"
 		(layer "F.Cu")
-		(at 138 93.75)
+		(at 124.6223 93.75)
 		(tags "T495X477K010ATE100 ")
 		(property "Reference" "REF**"
@@
 			(polygon
 				(pts
-					(xy 134.250808 91.650804) (xy 141.749192 91.650804) (xy 141.749192 92.449202) (xy 134.250808 92.449202)
+					(xy 120.873108 91.650804) (xy 128.371492 91.650804) (xy 128.371492 92.449202) (xy 120.873108 92.449202)
 				)
 			)
@@
 			(polygon
 				(pts
-					(xy 134.250808 95.050798) (xy 141.749192 95.050798) (xy 141.749192 95.849196) (xy 134.250808 95.849196)
+					(xy 120.873108 95.050798) (xy 128.371492 95.050798) (xy 128.371492 95.849196) (xy 120.873108 95.849196)
 				)
 			)
@@
 			(polygon
 				(pts
-					(xy 136.358804 92.449202) (xy 139.641196 92.449202) (xy 139.641196 95.050798) (xy 136.358804 95.050798)
-				)
-			)
+					(xy 122.981104 92.449202) (xy 126.263496 92.449202) (xy 126.263496 95.050798) (xy 122.981104 95.050798)
+				)
+			)
