File: PiZero_RTL_Panadapter.kicad_pcb (KiCad board)
At the start: 4 copper layers, 65 x 30 mm, 196 parts, among them J1 Conn_01x02, J2 JST GH 8 Position, J3 U.FL, J4 U.FL, J5 Conn_01x08, Q1 S8050T, Q2 BFS17, Q3 J310, Q4 BFS17, T1 DXW21BN2511NL, U1 RPM5.0-2.0, U10 SI5351B-B-GM1, U2 AP2114HA-3.3, U4 Raspberry Pi Zero 2W, U5 RTL2832U, U6 M24C02-WMN, U7 FE1.1s, U8 RTL8152B, U9 R820T2, Y1 25MHz

Commit message: PCB progress
Parts:
- moved Q1 2.14 mm to (148.4, 93.1), turned to 90 degrees
Routing:
- net /ETHERNET_25MHz_CLK: track 0.00 -> 51.2 mm, vias 0 -> 2
- net /USB-Ethernet Adapter/ETH_1V05: track 8.36 -> 18.1 mm
- net GND: track 250.1 -> 241.5 mm
- net Net-(Q1-C): track 26.3 -> 21.2 mm
- net /SDR/RTL_1V2: track 37.9 -> 39.4 mm
- net Net-(Q1-B): track 1.81 -> 3.21 mm
- net /RPI_I2C_SCL: track 64.6 -> 65.4 mm, vias 1 -> 3
- net /RPI_I2C_SDA: track 62.7 -> 63.4 mm, vias 1 -> 3
