File: PiZero_RTL_Panadapter.kicad_sch (KiCad schematic)
At the start: 15 parts, among them J2 Conn_01x02, J3 U.FL, J4 JST GH 8 Position, U1 Raspberry Pi Zero 2W, U11 RPM5.0-2.0, U2 AP2114H-3.3, U9 DXW21BN2511NL

Commit message: Schematic progress
Parts:
- added D3: RED, LED_SMD:LED_0402_1005Metric, symbol Device:LED_Filled
- added D6: BAV99, Package_TO_SOT_SMD:SOT-23, symbol Diode:BAV99
- added J5: U.FL, Connector_Coaxial:U.FL_Hirose_U.FL-R-SMT-1_Vertical, symbol Connector:Conn_Coaxial
- added R13: 1k, libraries:Worthington_R_0402, symbol Device:R_Small_US
- added R32: 0R, libraries:Worthington_R_0201, symbol Device:R_Small_US
- C89: DigiKey (none) -> 4713-GMC02CG102F25NTCT-ND; Manuyfacturer Part Number (none) -> GMC02CG102F25NT; Voltage (none) -> 25V
- D7: footprint (none) -> LED_SMD:LED_0402_1005Metric
- R47, R48, R71: footprint libraries:Worthington_R_0402 -> libraries:Worthington_R_0201
Connections:
- net +3V3: now also R71.1; no longer D7.2 (A)
- net +5V0: now also R13.1
- net GND: now also D7.1 (K), D3.1 (K), D6.1 (K), D6.2 (A), J5.2 (Ext), R32.1; no longer R71.2
- new net: D7.2 (A), R71.2
- new net: D3.2 (A), R13.2
- new net Clock Generator/EXT_CLK_OUT: D6.3 (K), J5.1 (In)
- new net Clock Generator/~{CLK_OUT_EN}: R32.2
- no-connect marks 6 -> 7
Other:
- sheet Clock Generator ports: added EXT_CLK_OUT, VCXO_IN, ~{CLK_OUT_EN}; removed none
- moved on the sheet: C65, D7, R71
