File: PiZero_RTL_Panadapter.kicad_sch (KiCad schematic)
At the start: 22 parts, among them J1 Conn_01x02, J2 JST GH 8 Position, J3 U.FL, J4 U.FL, J5 Conn_01x08, T1 DXW21BN2511NL, U1 RPM5.0-2.0, U2 AP2114HA-3.3, U4 Raspberry Pi Zero 2W

Commit message: PCB Layout finished?
Parts:
- T1: footprint libraries:DXW21BN2511NL -> libraries:XFMR_ATB2012-50011-T000
Connections:
- net GND: now also T1.1; no longer T1.2
- net IF_Q+: now also T1.3; no longer T1.4
- net IF_Q-: now also T1.4; no longer T1.3
- net at C3.2: now also T1.2; no longer T1.1
Changed lines of the file:
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@@
 			)
 		)
-		(property "Footprint" "libraries:DXW21BN2511NL"
+		(property "Footprint" "libraries:XFMR_ATB2012-50011-T000"
 			(at 204.47 208.28 0)
 			(hide yes)
