File: IF_Buffer.kicad_sch (KiCad schematic)
At the start: 18 parts, among them Q2 J310, Q3 BFS17

Commit message: Schematic progress
Parts:
- removed C27: 100n, libraries:Worthington_C_0402, symbol Device:C_Small
- removed C69, C72: 1n, libraries:Worthington_C_0402, symbol Device:C_Small
- removed Q3: BFS17, symbol Device:Q_NPN
- added C78, C94: 1n, libraries:Worthington_C_0402, symbol Device:C_Small
- added C83: 100n, libraries:Worthington_C_0201, symbol Device:C_Small
- added Q5: BFS17, Package_TO_SOT_SMD:SOT-23-3, symbol Device:Q_NPN
- C46: footprint libraries:Worthington_C_0402 -> libraries:Worthington_C_0201; DigiKey (none) -> 445-15903-1-ND; Manufacturer Part Number (none) -> C0603X6S1C104K030BC; Voltage (none) -> 16V
- C73: DigiKey (none) -> 4713-GMC02CG102F25NTCT-ND; Manufacturer Part Number (none) -> GMC02CG102F25NT; Voltage (none) -> 25V
- C84, C86: value 22p -> 22p, ±1%; DigiKey (none) -> 4713-GMC02CG220F50NTCT-ND; Manufacturer Part Number (none) -> GMC02CG220F50NT; Voltage (none) -> 50V
- C85: value 47p -> 47p, ±1%; DigiKey (none) -> 4713-GMC02CG470F50NTCT-ND; Manufacturer Part Number (none) -> GMC02CG470F50NT; Voltage (none) -> 50V
- L15, L16: value 100n -> 100n, ±2%
- Q2: footprint Package_TO_SOT_THT:TO-92_Inline -> Package_TO_SOT_SMD:SOT-23-3; DigiKey (none) -> MMBFJ310LT3GOSCT-ND; Manufacturer Part Number (none) -> MMBFJ310LT3G
Connections:
- net GND: now also C83.2
- net IF_IN: now also C78.1
- net at Q2.2 (S), R46.2: now also C94.1
- net at R49.1: now also C94.2, Q5.1 (B)
- net at Q2.3 (G), R45.2: now also C78.2
- net at R49.2, R50.1: now also C83.1, Q5.3 (C)
- net at C73.1, R52.2: now also Q5.2 (E)
Other:
- note added: "Targeting 73.095 MHz 1st RX IF for Kenwood TS-480/TS-850"
- note removed: "Targeting 73.095 MHz 1st RX IF for Kenwood TS-480"
- moved on the sheet: C73, C84, C85, L15

Commit message: Schematic and PCB progress
Parts:
- C82: renamed from C78; footprint libraries:Worthington_C_0402 -> libraries:Worthington_C_0201
- C84: renamed from C94; footprint libraries:Worthington_C_0402 -> libraries:Worthington_C_0201
- C86: renamed from C73; footprint libraries:Worthington_C_0402 -> libraries:Worthington_C_0201
- C87: renamed from C84; footprint Capacitor_SMD:C_0603_1608Metric_Pad1.08x0.95mm_HandSolder -> libraries:Worthington_C_0201
- C88: renamed from C85; footprint Capacitor_SMD:C_0603_1608Metric_Pad1.08x0.95mm_HandSolder -> libraries:Worthington_C_0201
- C89: renamed from C86; footprint Capacitor_SMD:C_0603_1608Metric_Pad1.08x0.95mm_HandSolder -> libraries:Worthington_C_0201
- R64: renamed from R45; footprint libraries:Worthington_R_0402 -> libraries:Worthington_R_0201
- R65: renamed from R51; footprint libraries:Worthington_R_0402 -> libraries:Worthington_R_0201
- R66: renamed from R46; footprint libraries:Worthington_R_0402 -> libraries:Worthington_R_0201
- R67: renamed from R49; footprint libraries:Worthington_R_0402 -> libraries:Worthington_R_0201
- R68: renamed from R50; footprint libraries:Worthington_R_0402 -> libraries:Worthington_R_0201
- R69: renamed from R52; footprint libraries:Worthington_R_0402 -> libraries:Worthington_R_0201
- renumbered C46 to C83, C83 to C85, L15 to L12, L16 to L13, Q2 to Q3, Q5 to Q4

Commit message: PCB Layout Progress
Parts:
- L12, L13: footprint libraries:Worthington_L_0603 -> libraries:Worthington_L_0603_RF
Other:
- note added: "CONSIDER REWORKING THIS TO USE MMBT5179"
Changed lines of the file:
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@@
 		)
 	)
+	(text "CONSIDER REWORKING THIS TO USE MMBT5179"
+		(exclude_from_sim no)
+		(at 171.45 147.32 0)
+		(effects
+			(font
+				(size 1.27 1.27)
+				(thickness 0.254)
+				(bold yes)
+			)
+			(justify left)
+		)
+	)
 	(text "Targeting 73.095 MHz 1st RX IF for Kenwood TS-480/TS-850"
 		(exclude_from_sim no)
@@
 			)
 		)
-		(property "Footprint" "libraries:Worthington_L_0603"
+		(property "Footprint" "libraries:Worthington_L_0603_RF"
 			(at 285.75 119.38 0)
 			(hide yes)
@@
 			)
 		)
-		(property "Footprint" "libraries:Worthington_L_0603"
+		(property "Footprint" "libraries:Worthington_L_0603_RF"
 			(at 321.31 119.38 0)
 			(hide yes)
