File: USB_HUB_FE1.1S.kicad_sch (KiCad schematic)
At the start: 13 parts, among them U5 FE1.1s

Commit message: Schematic progress
Parts:
- removed C31, C32, C33: 100n, libraries:Worthington_C_0402, symbol Device:C_Small
- removed C34: 10u, libraries:Worthington_C_0402, symbol Device:C_Small
- removed C35: 10u, libraries:Worthington_C_0603, symbol Device:C_Small
- removed D3: RED, symbol Device:LED_Filled
- removed R13: 1k, libraries:Worthington_R_0402, symbol Device:R_Small_US
- added C116, C117, C118, C93: 100n, libraries:Worthington_C_0201, symbol Device:C_Small
- added C119, C54: 10u, libraries:Worthington_C_0402, symbol Device:C_Small
Connections:
- net 12.0MHz_CLK_IN: now also C93.2; no longer R44.2, U5.3 (XIN/12MHz)
- net 5V0_IN: now also C116.1
- net GND: now also C116.2, C117.2, C118.2, C119.2, C54.2
- net HUB_1V8: now also C117.1, C54.1
- net HUB_3V3: now also C118.1, C119.1
- new net: C93.1, R44.2, U5.3 (XIN/12MHz)

Commit message: Schematic and PCB progress
Parts:
- R20: renamed from R14; footprint libraries:Worthington_R_0402 -> libraries:Worthington_R_0201
- R21: renamed from R44; footprint libraries:Worthington_R_0402 -> libraries:Worthington_R_0201
- R22: renamed from R15; footprint libraries:Worthington_R_0402 -> libraries:Worthington_R_0201
- R23: renamed from R16; footprint libraries:Worthington_R_0402 -> libraries:Worthington_R_0201
- R24: renamed from R17; footprint libraries:Worthington_R_0402 -> libraries:Worthington_R_0201
- renumbered C116 to C28, C117 to C29, C118 to C30, C54 to C31, C119 to C32, C93 to C33, U5 to U7
Connections:
- net USB1_N renamed USB1_90R_N
- net USB1_P renamed USB1_90R_P
- net USB2_N renamed USB2_90R_N
- net USB2_P renamed USB2_90R_P
- net USB3_N renamed USB3_90R_N
- net USB3_P renamed USB3_90R_P
- net USB4_N renamed USB4_90R_N
- net USB4_P renamed USB4_90R_P
- net USBUP_DM renamed USBUP_90R_N
- net USBUP_DP renamed USBUP_90R_P
Other:
- note added: "Integrated USB Pull-Ups"
- moved on the sheet: R22, R23, R24

Commit message: PCB Layout Progress
Other:
- note added: "REVIEW HOW OVCJ OVERCURRENT WORKS"
Changed lines of the file:
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@@
 	(generator_version "10.0")
 	(paper "B")
+	(text "REVIEW HOW OVCJ OVERCURRENT WORKS"
+		(exclude_from_sim no)
+		(at 226.314 147.32 0)
+		(effects
+			(font
+				(size 1.27 1.27)
+			)
+		)
+	)
 	(text "90-Ohm Differential Impedance"
 		(exclude_from_sim no)
