File: HF_Frontend.kicad_sch (KiCad schematic)
At the start: 7 parts

Commit message: Schematic progress
Parts:
- removed L12: 330n, libraries:Worthington_L_0603, symbol Device:L_Small
- added C74: 82p, libraries:Worthington_C_0402, symbol Device:C_Small
- added C87: 100n, libraries:Worthington_C_0402, symbol Device:C_Small
- added C88: 1n, libraries:Worthington_C_0402, symbol Device:C_Small
- added L17: 180n, libraries:Worthington_L_0603, symbol Device:L_Small
- added L21: 470n, libraries:Worthington_L_0603, symbol Device:L_Small
- added Q4: BFS17, symbol Device:Q_NPN
- added R53, R55: π1, libraries:Worthington_R_0402, symbol Device:R_Small_US
- added R54: π2, libraries:Worthington_R_0402, symbol Device:R_Small_US
- added R63: 1k, libraries:Worthington_R_0402, symbol Device:R_Small_US
- added R64: 180, libraries:Worthington_R_0402, symbol Device:R_Small_US
- added R65: 270, libraries:Worthington_R_0402, symbol Device:R_Small_US
- added R66: 680, libraries:Worthington_R_0402, symbol Device:R_Small_US
- added R67: 10, libraries:Worthington_R_0402, symbol Device:R_Small_US
- C80: value 68p -> 82p; footprint Capacitor_SMD:C_0603_1608Metric_Pad1.08x0.95mm_HandSolder -> libraries:Worthington_C_0402
- C81: value 150p -> 82p
- C82: value 150p -> 220p
- C83: value 68p -> 1n; footprint Capacitor_SMD:C_0603_1608Metric_Pad1.08x0.95mm_HandSolder -> libraries:Worthington_C_0402
- L13: value 390n -> 470n; Murata LQW18ANR39G00D -> LQW18ANR47G00D; Self-Resonance (none) -> 700 MHz
- L14: value 330n -> 470n; Murata LQW18ANR33G00D -> LQW18ANR47G00D; Self-Resonance (none) -> 700 MHz
Connections:
- net GND: now also C87.2, C88.2, L17.1, L21.1, R53.1, R55.1, R64.1, R66.1; no longer C80.2, C83.2
- net at C80.1: now also C74.2, L17.2
- net <25MHz_OUT: now reaches C81.1, L13.2
- net 28.8MHz_OUT: no longer names the net of C83.1
- net 28.8MHz_OUT: now also R54.2, R55.2; no longer L14.1
- new net: C83.2, Q4.1 (B), R63.1, R66.2
- new net: Q4.2 (E), R67.2
- new net: C74.1, L14.1, Q4.3 (C), R65.1
- new net: C88.1, R64.2, R67.1
- new net >25MHz_OUT: C80.2, L21.2
- new net IF_IN: R53.2, R54.1
- new net VCC_IN: C87.1, R63.2, R65.2
Other:
- note added: "25 MHz High-Pass"
- note added: "25 MHz Low-Pass"
- note added: "Common Emitter ~8dB Gain"
- note added: "Diplexer ~25 MHz Cutoff Frequency"
- note added: "π Attenuator"
- note removed: "7th Order Chebyshev Lowpass"
- note removed: "Targeting 28.8 MHz Clock for RTL2832U"
- note removed: "~30 MHz Cutoff Frequency"
- moved on the sheet: C81, C82, L13, L14

Commit message: Schematic progress
Parts:
- removed C81: 82p, Capacitor_SMD:C_0603_1608Metric_Pad1.08x0.95mm_HandSolder, symbol Device:C_Small
- removed C83: 1n, libraries:Worthington_C_0402, symbol Device:C_Small
- removed Q4: BFS17, symbol Device:Q_NPN
- added C122: 220p, ±1%, libraries:Worthington_C_0201, symbol Device:C_Small
- added C95: 1n, libraries:Worthington_C_0402, symbol Device:C_Small
- added Q6: BFS17, Package_TO_SOT_SMD:SOT-23-3, symbol Device:Q_NPN
- C74, C80: value 82p -> 82p, ±1%; DigiKey (none) -> 4713-GMC02CG820F50NTCT-ND; Manufacturer Part Number (none) -> GMC02CG820F50NT
- C82: value 220p -> 220p, ±1%; footprint Capacitor_SMD:C_0603_1608Metric_Pad1.08x0.95mm_HandSolder -> libraries:Worthington_C_0201; DigiKey (none) -> 4713-GMC02CG221F50NTCT-ND; Manufacturer Part Number (none) -> GMC02CG221F50NT; Voltage (none) -> 50V
- C87: footprint libraries:Worthington_C_0402 -> libraries:Worthington_C_0201; DigiKey (none) -> 445-15903-1-ND; Manufacturer Part Number (none) -> C0603X6S1C104K030BC; Voltage (none) -> 16V
- C88: DigiKey (none) -> 4713-GMC02CG102F25NTCT-ND; Manuyfacturer Part Number (none) -> GMC02CG102F25NT; Voltage (none) -> 25V
- L13, L14, L21: value 470n -> 470n, ±2%
- L17: value 180n -> 180n, ±2%
Connections:
- net <25MHz_OUT: now also C122.1
- net GND: now also C122.2
- net at R54.2, R55.2: now also C95.1
- net at R63.1, R66.2: now also C95.2, Q6.1 (B)
- net at R67.2: now also Q6.2 (E)
- net at C74.1, L14.1, R65.1: now also Q6.3 (C)
Other:
- moved on the sheet: C82, L13, L17, L21, R63

Commit message: Schematic and PCB progress
Parts:
- C75: renamed from C95; footprint libraries:Worthington_C_0402 -> libraries:Worthington_C_0201
- C76: renamed from C88; footprint libraries:Worthington_C_0402 -> libraries:Worthington_C_0201
- R56: renamed from R53; footprint libraries:Worthington_R_0402 -> libraries:Worthington_R_0201
- R57: renamed from R54; footprint libraries:Worthington_R_0402 -> libraries:Worthington_R_0201
- R58: renamed from R55; footprint libraries:Worthington_R_0402 -> libraries:Worthington_R_0201
- R59: renamed from R63; footprint libraries:Worthington_R_0402 -> libraries:Worthington_R_0201
- R60: renamed from R66; footprint libraries:Worthington_R_0402 -> libraries:Worthington_R_0201
- R61: renamed from R65; footprint libraries:Worthington_R_0402 -> libraries:Worthington_R_0201
- R62: renamed from R67; footprint libraries:Worthington_R_0402 -> libraries:Worthington_R_0201
- R63: renamed from R64; footprint libraries:Worthington_R_0402 -> libraries:Worthington_R_0201
- renumbered C87 to C77, C74 to C78, C82 to C79, C122 to C81, L13 to L10, L21 to L11, L14 to L8, L17 to L9, Q6 to Q2

Commit message: PCB Layout Progress
Parts:
- C78, C80: footprint libraries:Worthington_C_0402 -> libraries:Worthington_C_0201
- L10, L11, L8, L9: footprint libraries:Worthington_L_0603 -> libraries:Worthington_L_0603_RF
Connections:
- net PRE_AMP_OUT-DIPLEXER_IN: now reaches C78.1, L8.1, Q2.3 (C), R61.1
Other:
- note added: "CONSIDER REWORKING THIS TO USE MMBT5179"
Changed lines of the file:
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@@
 		)
 	)
+	(text "CONSIDER REWORKING\nTHIS TO USE MMBT5179"
+		(exclude_from_sim no)
+		(at 226.568 114.554 0)
+		(effects
+			(font
+				(size 1.27 1.27)
+				(thickness 0.254)
+				(bold yes)
+			)
+			(justify right)
+		)
+	)
 	(text "Diplexer ~25 MHz Cutoff Frequency"
 		(exclude_from_sim no)
@@
 		)
 	)
+	(label "PRE_AMP_OUT-DIPLEXER_IN"
+		(at 240.03 96.52 0)
+		(effects
+			(font
+				(size 1.27 1.27)
+			)
+			(justify left bottom)
+		)
+	)
 	(hierarchical_label "<25MHz_OUT"
 		(shape output)
@@
 			)
 		)
-		(property "Footprint" "libraries:Worthington_C_0402"
+		(property "Footprint" "libraries:Worthington_C_0201"
 			(at 337.82 80.01 0)
 			(hide yes)
@@
 			)
 		)
-		(property "Footprint" "libraries:Worthington_C_0402"
+		(property "Footprint" "libraries:Worthington_C_0201"
 			(at 297.18 80.01 0)
 			(hide yes)
@@
 			)
 		)
-		(property "Footprint" "libraries:Worthington_L_0603"
+		(property "Footprint" "libraries:Worthington_L_0603_RF"
 			(at 358.14 87.63 0)
 			(hide yes)
@@
 			)
 		)
-		(property "Footprint" "libraries:Worthington_L_0603"
+		(property "Footprint" "libraries:Worthington_L_0603_RF"
 			(at 297.18 113.03 0)
 			(hide yes)
@@
 			)
 		)
-		(property "Footprint" "libraries:Worthington_L_0603"
+		(property "Footprint" "libraries:Worthington_L_0603_RF"
 			(at 317.5 87.63 0)
 			(hide yes)
@@
 			)
 		)
-		(property "Footprint" "libraries:Worthington_L_0603"
+		(property "Footprint" "libraries:Worthington_L_0603_RF"
 			(at 337.82 113.03 0)
 			(hide yes)

Commit message: Small PCB layout tweaks
Beautification, if you will...
Parts:
- C76: Manufacturer Part Number (none) -> GMC02CG102F25NT; Manuyfacturer Part Number GMC02CG102F25NT -> (none)
Changed lines of the file:
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@@
 			)
 		)
-		(property "Manuyfacturer Part Number" "GMC02CG102F25NT"
+		(property "Manufacturer Part Number" "GMC02CG102F25NT"
 			(at 218.694 135.636 0)
 			(show_name no)
