File: Modules/PWR_RPM5.0_AP2114/PWR_RPM5.0_AP2114.kicad_pcb (KiCad board)
At the start: 4 copper layers, 39.8 x 52.7 mm, 28 parts, among them J1 Screw Terminal, J5 2.54 Pins, J6 2.54 Pins, J8 Red/Black PowerPole 45, J9 2.54mm Header, SW1 SW_SP3T, SW2 SPST, U1 RPM5.0-2.0, U2 AP2114HA-3.3

Commit message: Added silkscreen art to PCB
Labels on bottom side, primarily
Parts:
- added G***: LOGO, libraries:Logo_10mm_inv, B.Cu at (177.2, 87.6)
- D1: value RED -> AMBER
Other:
- board text added: "+6-17V"
- board text added: "3V3/1A"
- board text added: "5V/2A"

Commit message: PCB tweaks, generated gerbers
Parts:
- added J8: Red/Black PowerPole 45, libraries:APP_ASMPR45-1X2-RK, B.Cu at (161.1, 101.9)
- C11, C13, C9: value 1u -> 10u
- C5, C7, C8: footprint Capacitor_THT:CP_Radial_D8.0mm_P2.50mm -> Capacitor_THT:CP_Radial_D6.3mm_P2.50mm
- R1, R4: value 1k -> 3k
- R5: value 1k -> 1k3
- RV1: footprint Potentiometer_THT:Potentiometer_Runtron_RM-065_Vertical -> Potentiometer_THT:Potentiometer_Bourns_3299Y_Vertical
- moved C5 8.69 mm to (160.1, 64.9)
- moved RV1 6.71 mm to (159.5, 77.3)
- moved J1 4.28 mm to (161.9, 70.3), turned to -90 degrees
- moved C7 2.07 mm to (168.9, 64.9), turned to 0 degrees
- moved C8 1.94 mm to (177.7, 64.9), turned to 0 degrees
- moved G*** 1.02 mm to (176.1, 87.6)
- moved J8 0.10 mm to (169.0, 101.9)
- turned R3 to 0 degrees
Routing:
- net Net-(RV1-Pad3): track 17.2 -> 12.4 mm
- net Net-(J9-Pin_3): track 33.9 -> 36.6 mm
- net Net-(U1-Trim): track 15.8 -> 18.0 mm
- net Net-(R3-Pad2): track 5.11 -> 6.29 mm
- net GND: track 151.2 -> 152.3 mm, vias 30 -> 31
- net /PWR_IN: track 29.1 -> 29.8 mm
Other:
- board size 39.8 x 52.7 mm -> 39.9 x 52.7 mm
- board text added: "5"
- board text added: "MΩ"
- board text added: "Rev A"
- board text added: "VIN"
- board text added: "VOUT SENSE"
- board text removed: "+12V"
- board text removed: "SENSE"
