File: Modules/PWR_RPM5.0_AP2114/PWR_RPM5.0_AP2114.kicad_sch (KiCad schematic)
At the start: 28 parts, among them J1 Screw Terminal, J5 2.54 Pins, J6 2.54 Pins, J8 Red/Black PowerPole 45, J9 2.54mm Header, SW1 SW_SP3T, SW2 SPST, U1 RPM5.0-2.0, U2 AP2114HA-3.3

Commit message: PCB tweaks, generated gerbers
Parts:
- C10, C12, C6: DigiKey 399-5279-1-ND -> 4713-GMC31X5R226M25NTCT-ND; ESR 6Ω -> (none); Manufacturer Part Number T491A336K010AT -> (none); Part Number (none) -> GMC31X5R226M25NT; Voltage 50V -> 25V
- C11, C13: value 1u -> 10u; Manufacturer Part Number T491A336K010AT -> GMC10X5R106K25NT
- C5, C7, C8: footprint Capacitor_THT:CP_Radial_D8.0mm_P2.50mm -> Capacitor_THT:CP_Radial_D6.3mm_P2.50mm
- C9: value 1u -> 10u; DigiKey 399-5279-1-ND -> 4713-GMC10X5R106K25NTCT-ND; ESR 6Ω -> (none); Manufacturer Part Number T491A336K010AT -> (none); Part Number (none) -> GMC10X5R106K25NT
- D1: DigiKey (none) -> 160-1968-ND; Part Number (none) -> LTL-4291N
- D2: DigiKey (none) -> 5366-LLR3ED199G-ND; Part Number (none) -> LLR3ED199G
- D3: DigiKey (none) -> BL-BGE1V5D-AT-ND; Part Number (none) -> BL-BGE1V5D-AT
- J1: DigiKey (none) -> 277-1273-ND; Part Number (none) -> 1725656
- J8: DigiKey (none) -> 2243-ASMPR45-1X2-RK-ND; Part Number (none) -> ASMPR45-1X2-RK
- R1, R4: value 1k -> 3k; DigiKey (none) -> 4713-RM04F3001CT-ND; Part Number (none) -> RM04F3001CT
- R3: DigiKey (none) -> 4713-RM04F9531CT-ND; Part Number (none) -> RM04F9531CT
- R5: value 1k -> 1k3; DigiKey (none) -> 4713-RM04F1301CT-ND; Part Number (none) -> RM04F1301CT
- R6: DigiKey (none) -> 4713-RM04F3403CT-ND; Part Number (none) -> RM04F3403CT
- RV1: footprint Potentiometer_THT:Potentiometer_Runtron_RM-065_Vertical -> Potentiometer_THT:Potentiometer_Bourns_3299Y_Vertical; DigiKey (none) -> 3299Y-505LF-ND; Part Number (none) -> 3299Y-1-505LF
- SW1: DigiKey (none) -> CKN9561-ND; Part Number (none) -> OS103011MA7QP1
- SW2: DigiKey (none) -> CKN9559-ND; Part Number (none) -> OS102011MA1QN1
- U1: DigiKey (none) -> 945-3455-ND; Part Number (none) -> RPM5.0-2.0-CT
- U2: DigiKey (none) -> AP2114HA-3.3TRG1DICT-ND; Part Number (none) -> AP2114HA-3.3TRG1

Commit message: Corrected breadboard width
Gave me a chance to rearrange some of the 3V3 stuff, looks much healthier now
Parts:
- S1: footprint Connector_PinHeader_1.00mm:PinHeader_1x01_P1.00mm_Horizontal -> libraries:Breadboard_400
Changed lines of the file:
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@@
 			)
 		)
-		(property "Footprint" "Connector_PinHeader_1.00mm:PinHeader_1x01_P1.00mm_Horizontal"
+		(property "Footprint" "libraries:Breadboard_400"
 			(at 266.7 143.51 0)
 			(hide yes)
