File: Modules/ClockGen_Si5351X_QFN16/ClockGen_Si5351X_QFN16.kicad_sch (KiCad schematic)
At the start: 0 parts

Commit message: Started Si5351 module
Parts:
- added C1, C11, C12, C13, C14, C15, C17, C18, C19, C20, C21, C23, C24, C25, C26, C28, C29, C3, C30, C31: 0402, libraries:Worthington_C_0402, symbol Device:C_Small
- added C10: 10u, libraries:Worthington_C_0402, symbol Device:C_Small
- added C2: 1u, libraries:Worthington_C_0402, symbol Device:C_Small
- added C4, C5, C7, C8, C9: 100n, libraries:Worthington_C_0201, symbol Device:C_Small
- added C6: 47u, libraries:Worthington_C_0805, symbol Device:C_Small
- added J1: 2.54mm Header, Connector_PinHeader_2.54mm:PinHeader_1x04_P2.54mm_Horizontal, symbol Connector_Generic:Conn_01x04
- added J2, J3, J4, J5, J7: Conn_Coaxial, Connector_Coaxial:SMA_Molex_73251-2200_Horizontal, symbol Connector:Conn_Coaxial
- added L1, L10, L11, L12, L13, L15, L16, L17, L18, L20, L3, L4, L5, L6, L7, L9: 0603, libraries:Worthington_L_0603_RF, symbol Device:L_Small
- added Q1: Q_NMOS_DGS, Package_TO_SOT_SMD:SOT-523, symbol Transistor_FET:Q_NMOS_GSD
- added R1, R2: 4k7, libraries:Worthington_R_0201, symbol Device:R_Small_US
- added R3, R4, R5, R6: 0R, libraries:Worthington_R_0402, symbol Device:R_US
- added SW1: SW_SPDT, symbol Switch:SW_SPDT
- added U1: NCV68061, Package_SO:TSOP-6_1.65x3.05mm_P0.95mm, symbol Power_Management:LM66100DCK
- added U2: NCP361SN, Package_SO:TSOP-5_1.65x3.05mm_P0.95mm, symbol Power_Protection:NCP349MNAE
- added U3: SI5351B-B-GM1, Package_DFN_QFN:QFN-16-1EP_3x3mm_P0.5mm_EP1.45x1.45mm, symbol Oscillator:Si5351A-B-GT
- added U4: AP2114HA-3.3, Package_TO_SOT_SMD:SOT-223, symbol Regulator_Linear:AP2112K-3.3
- added Y1: 25MHz, libraries:Crystal_SMD_Kyocera_CX3225SB-4Pin_3.2x2.5mm, symbol Device:Crystal_GND24
Connections:
- new net: C10.1, C4.1, C5.1, C6.1, C7.1, C8.1, C9.1, J1.1 (Pin_1), R1.2, R2.2, SW1.1 (A), U3.11 (VDDOD), U3.14 (VDDOC), U3.16 (VDD), U3.8 (VDDOB), U3.9 (VDDOA), U4.2 (VOUT)
- new net: C24.1, L10.2, L16.1
- new net: C23.1, C28.1, L15.2, L9.2
- new net: C28.2, L18.1
- new net: C13.2, L1.2
- new net: C2.1, Q1.3 (D), U1.4 (D), U2.1 (IN), U2.7 (IN)
- new net: U2.4 (OUT), U2.5 (OUT), U4.3 (VIN)
- new net: C17.2, L9.1
- new net: C18.1, L10.1, L4.2
- new net: C14.2, C20.1, L6.2
- new net: C26.2, C30.1, L17.2
- new net: J1.3 (Pin_3), R2.1, U3.4 (SCL)
- new net: J1.4 (Pin_4), R1.1, U3.5 (SDA)
- new net: C3.1, U3.2 (XB), Y1.1
- new net: C1.1, U3.1 (XA), Y1.3
- new net: C15.2, C19.1, C21.1, L11.1, L5.2
- new net: C19.2, L7.2
- new net: Q1.2 (S), U1.3 (EN), U1.6 (S)
- new net: Q1.1 (G), U1.5 (G)
- new net: C20.2, C26.1, L12.2
- new net: C25.2, L13.2
- new net CLK0: C11.1, C17.1, L3.2, R3.2
- new net CLK0_BANDPASS: C31.1, J3.1 (In), L18.2, L20.2
- new net CLK0_T: R3.1, U3.10 (CLK0)
- new net CLK1: C12.1, L4.1, R4.2
- new net CLK1_LOWPASS: C29.1, J4.1 (In), L16.2
- new net CLK1_T: R4.1, U3.7 (CLK1)
- new net CLK2: C13.1, C15.1, L5.1, R5.2
- new net CLK2_BANDSTOP: C21.2, C25.1, J5.1 (In), L11.2
- new net CLK2_T: R5.1, U3.13 (CLK2)
- new net CLK3: C14.1, R6.2
- new net CLK3_HIGHPASS: C30.2, J7.1 (In)
- new net CLK3_T: R6.1, U3.12 (CLK3)
- new net GND: C1.2, C10.2, C11.2, C12.2, C18.2, C2.2, C23.2, C24.2, C29.2, C3.2, C31.2, C4.2, C5.2, C6.2, C7.2, C8.2, C9.2, J1.2 (Pin_2), J2.2 (Ext), J3.2 (Ext), J4.2 (Ext), J5.2 (Ext), J7.2 (Ext), L1.1, L12.1, L13.1, L15.1, L17.1, L20.1, L3.1, L6.1, L7.1, SW1.3 (C), U1.2 (GND), U2.2 (GND), U2.6 (~{EN}), U3.15 (GND), U3.17 (GND), U4.1 (GND), U4.4 (GND), Y1.2 (G), Y1.4 (G)
- new net VCXO_IN: J2.1 (In), U3.3 (VC)
- new net ~{OUTPUT_EN}: SW1.2 (B), U3.6 (~{OEB})
Other:
- note added: "5th Order Chebyshev Bandpass"
- note added: "5th Order Chebyshev Bandstop"
- note added: "7th Order Chebyshev Diplexer"
- note added: "7th Order Chebyshev Lowpass"
- note added: "Overvoltage Protection"
- note added: "Reverse Polarity Protection"
- note added: "Si5351 Features Selectable Internal Capacitors External Load Capacitors Likely Unnecessary"

Commit message: Rev A of schematic completed
Parts:
- removed R1: 4k7, libraries:Worthington_R_0201, symbol Device:R_Small_US
- removed U4: AP2114HA-3.3, Package_TO_SOT_SMD:SOT-223, symbol Regulator_Linear:AP2112K-3.3
- added C10, C11, C12, C33, C34, C35, C36, C9: 2u2, libraries:Worthington_C_0402, symbol Device:C_Small
- added D1, D2: ESDSLC5V0, Diode_SMD:D_SOD-882, symbol Diode:ESD9B3.3ST5G
- added D3, D6, D7, D8, D9: SLZST311N10, Diode_SMD:D_SOD-882, symbol Diode:ESD9B3.3ST5G
- added D4: 1N5819W, Diode_SMD:D_SOD-123F, symbol Device:D_Schottky
- added D5: RED, libraries:Worthington_LED_0402, symbol Device:LED_Filled
- added H1, H2, H3, H4: M2.5, MountingHole:MountingHole_2.7mm_M2.5_ISO7380_Pad, symbol Mechanical:MountingHole_Pad
- added J7, J8: 2.54 Pins, Connector_PinHeader_2.54mm:PinHeader_2x02_P2.54mm_Vertical, symbol Connector_Generic:Conn_01x04
- added Q2: GSFK0502, Package_TO_SOT_SMD:SOT-363_SC-70-6, symbol Transistor_FET:Q_Dual_NMOS_S1G1D2S2G2D1
- added R1: 0R, libraries:Worthington_R_0402, symbol Device:R_US
- added R3: 1k, libraries:Worthington_R_0402, symbol Device:R_Small_US
- added R8: 1k3, libraries:Worthington_R_0201, symbol Device:R_Small_US
- added RN1: 4k7, libraries:RESCAXE80P320X160X70-8N, symbol Libraries:R_Network04_Split
- added U4: SL6206-ADJ, Package_TO_SOT_SMD:SOT-23-5, symbol Regulator_Linear:SPX3819M5-L
- J2, J3, J4, J5: value Conn_Coaxial -> SMA
- J6: renamed from J7; value Conn_Coaxial -> SMA
- Q1: value Q_NMOS_DGS -> GSF0301; DigiKey (none) -> 4786-GSF0301CT-ND; Part Number (none) -> GSF0301
- R2: value 4k7 -> 2k8; footprint libraries:Worthington_R_0201 -> libraries:Worthington_R_0402
- SW1: footprint (none) -> Button_Switch_THT:SW_Slide_SPDT_Angled_CK_OS102011MA1Q
- U1: DigiKey (none) -> 488-NCV68061SNAIT1GCT-ND; Field6 (none) -> NCV68061SNAIT1G
- renumbered C2 to C1, C9 to C13, C10 to C14, C11 to C15, C12 to C16, C13 to C17, C14 to C18, C15 to C19, C1 to C2, C17 to C20, C18 to C21, C19 to C22, C20 to C23, C21 to C24, C23 to C25, C24 to C26, C25 to C27, C26 to C28, C28 to C29, C29 to C30, C30 to C31, C31 to C32, L12 to L10, L13 to L11, L15 to L12, L16 to L13, L17 to L14, L18 to L15, L20 to L16, L3 to L2, L4 to L3, L5 to L4, L6 to L5, L7 to L6, L9 to L7, L10 to L8, L11 to L9, R3 to R4, R4 to R5, R5 to R6, R6 to R7
Connections:
- net CLK0: now also C9.2; no longer R4.2
- net CLK0_BANDPASS: now also C33.2, D6.2 (A2); no longer C32.1, L15.2, L16.2
- net CLK1: now also C10.2; no longer R5.2
- net CLK1_LOWPASS: now also C34.2, D7.2 (A2); no longer C30.1, L13.2
- net CLK2: now also C11.2; no longer R6.2
- net CLK2_BANDSTOP: now also C35.2, D8.2 (A2); no longer C24.2, C27.1, L9.2
- net CLK3: now also C12.2; no longer R7.2
- net CLK3_HIGHPASS: now also C36.2, D9.2 (A2); no longer C31.2
- net GND: now also J1.1 (Pin_1), D1.2 (A2), D2.1 (A1), D3.1 (A1), D6.1 (A1), D7.1 (A1), D8.1 (A1), D9.1 (A1), H1.1, H2.1, H3.1, H4.1, J7.1 (Pin_1), J7.3 (Pin_3), J8.1 (Pin_1), J8.3 (Pin_3), R3.1, R8.2, U4.2 (GND); no longer J1.2 (Pin_2)
- net VCXO_IN: now also D3.2 (A2), R1.1; no longer U3.3 (VC)
- net +3V3: now reaches C13.1, C14.1, C4.1, C5.1, C6.1, C7.1, C8.1, R2.2, SW1.1 (A), U3.11 (VDDOD), U3.14 (VDDOC), U3.16 (VDD), U3.8 (VDDOB), U3.9 (VDDOA)
- net +3V3: now also D5.2 (A), Q2.2 (G), Q2.5 (G), RN1.2, RN1.3, U4.5 (OUT); no longer J1.1 (Pin_1)
- net +5V: now reaches U2.4 (OUT), U2.5 (OUT)
- net +5V: now also D4.2 (A), U4.1 (IN), U4.3 (EN)
- net I2C_SCL_5V: now reaches J1.4 (Pin_4)
- net I2C_SCL_5V: now also D1.1 (A1), Q2.3 (D), RN1.5; no longer U3.5 (SDA)
- net VCC: now reaches Q1.2 (S), U1.3 (EN), U1.6 (S)
- net VCC: now also J1.2 (Pin_2), J7.2 (Pin_2), J7.4 (Pin_4), J8.2 (Pin_2), J8.4 (Pin_4)
- new net: C30.1, C34.1, L13.2
- new net: C10.1, R5.2
- new net: D5.1 (K), R8.1
- new net: R2.1, R3.2, U4.4 (ADJ)
- new net: C12.1, R7.2
- new net: C11.1, R6.2
- new net: C31.2, C36.1
- new net: C24.2, C27.1, C35.1, L9.2
- new net: C32.1, C33.1, L15.2, L16.2
- new net: C9.1, R4.2
- new net +5V_PROTECT: D4.1 (K), RN1.1 (4), RN1.4
- new net I2C_SCL: Q2.4 (S), RN1.6, U3.4 (SCL)
- new net I2C_SDA: Q2.1 (S), RN1.7 (5), U3.5 (SDA)
- new net I2C_SDA_5V: D2.2 (A2), J1.3 (Pin_3), Q2.6 (D), RN1.8
- new net VCXO_IN_T: R1.2, U3.3 (VC)
Other:
- note added: "3V3 LDO"
- note added: "5th Order Bandpass"
- note added: "5th Order Bandstop"
- note added: "7th Order Highpass"
- note added: "7th Order Lowpass"
- note removed: "5th Order Chebyshev Bandpass"
- note removed: "5th Order Chebyshev Bandstop"
- note removed: "7th Order Chebyshev Diplexer"
- note removed: "7th Order Chebyshev Lowpass"
- moved on the sheet: C1, C13, C14, C15, C16, C17, C18, C19, C2, C20, C21, C22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

Commit message: Added support for Si5351A and Si5351C
Quite a clever setup, if I do say so myself
Parts:
- removed Q1: GSF0301, Package_TO_SOT_SMD:SOT-523, symbol Transistor_FET:Q_NMOS_GSD
- removed R1: 0R, libraries:Worthington_R_0402, symbol Device:R_US
- removed U2: NCP361SN, Package_SO:TSOP-5_1.65x3.05mm_P0.95mm, symbol Power_Protection:NCP349MNAE
- added C38, C4: 1u, libraries:Worthington_C_0402, symbol Device:C_Small
- added D6: 1N5819W, Diode_SMD:D_SOD-123F, symbol Device:D_Schottky
- added J1: Screw Terminal, TerminalBlock_Phoenix:TerminalBlock_Phoenix_MPT-0,5-2-2.54_1x02_P2.54mm_Horizontal, symbol Connector:Screw_Terminal_01x02
- added JP1, JP2: Jumper_3_Bridged12, symbol Jumper:Jumper_3_Bridged12
- added Q3: GSFJ0300, Package_TO_SOT_SMD:SOT-563, symbol Transistor_FET:Q_Dual_NMOS_S1G1D2S2G2D1
- added R11: 0R, libraries:Worthington_R_0402, symbol Device:R_US
- added R12, R13: 1k, libraries:Worthington_R_0201, symbol Device:R_Small_US
- added R2: 1k, libraries:Worthington_R_0402, symbol Device:R_Small_US
- added R3: 5k83, libraries:Worthington_R_0402, symbol Device:R_Small_US
- added S1: Breadboard 3D Model, Connector_PinHeader_1.00mm:PinHeader_1x01_P1.00mm_Horizontal, symbol Graphic:SYM_Arrow45_Small
- added U2: NCP718BSNADJ, Package_TO_SOT_SMD:SOT-23-5, symbol Regulator_Linear:NCP718xSN500
- added U5: NCV68261, Package_SO:TSOP-6_1.65x3.05mm_P0.95mm, symbol Power_Management:LM66100DCK
- J2: renamed from J1; value 2.54mm Header -> JST SH; footprint Connector_PinHeader_2.54mm:PinHeader_1x04_P2.54mm_Horizontal -> Connector_JST:JST_SH_SM04B-SRSS-TB_1x04-1MP_P1.00mm_Horizontal
- RN1: value 4k7 -> 1k0
- U1: value NCV68061 -> NCV68261
- U4: value SL6206-ADJ -> AP2127K-ADJ; DigiKey 5399-SL6206-ADJMRCT-ND -> AP2127K-ADJTRG1DICT-ND; PSRR (none) -> 68dB @ 1kHz; Part Number SL6206-ADJMR -> AP2127K-ADJTRG1; V_{DROPOUT} (none) -> 220mV @ 300mA, 60°C; V_{IN, Max} (none) -> +6V
- renumbered C6 to C13, C13 to C14, C14 to C15, C15 to C16, C16 to C17, C17 to C18, C18 to C19, C19 to C20, C20 to C21, C21 to C22, C22 to C23, C23 to C24, C24 to C25, C25 to C26, C26 to C27, C27 to C28, C28 to C29, C29 to C30, C30 to C31, C31 to C32, C32 to C33, C33 to C34, C34 to C35, C35 to C36, C36 to C37, C4 to C5, C5 to C6, D8 to D10, D9 to D11, D1 to D2, D2 to D3, D3 to D4, D4 to D5, D5 to D7, D6 to D8, D7 to D9, J7 to J3, J2 to J4, J8 to J5, J3 to J6, J4 to J7, J5 to J8, J6 to J9, R8 to R10, R2 to R4, R3 to R5, R4 to R6, R5 to R7, R6 to R8, R7 to R9
Connections:
- net +5V: now also D5.1 (K), J3.2 (Pin_2), J3.4 (Pin_4), C38.1, C4.1, Q3.3 (D), U5.3 (D); no longer D5.2 (A)
- net GND: now also U1.5 (GND), C38.2, C4.2, J1.1 (Pin_1), R13.2, R3.1, U2.2 (GND), U5.5 (GND); no longer U1.2 (GND)
- net VCC: now also U1.1 (S), U1.4 (EN), J1.2 (Pin_2), Q3.1 (S); no longer J2.2 (Pin_2), J3.2 (Pin_2), J3.4 (Pin_4), J5.2 (Pin_2), J5.4 (Pin_4), U1.3 (EN)
- net ~{OUTPUT_EN}: now also JP1.1 (A), JP2.3 (B); no longer U3.6 (~{OEB})
- net at C1.1: now also J2.2 (Pin_2), U1.3 (D), Q3.6 (D), U2.1 (IN), U2.3 (EN); no longer U1.4 (D)
- net +3V3 renamed +3V0
- net +3V0: now also R12.1
- net +5V_PROTECT renamed +5V_I2C_PULLUP
- net +5V_I2C_PULLUP: now also D6.1 (K); no longer D5.1 (K)
- net VCXO_IN renamed VCXO_IN/CLK_IN
- net VCXO_IN/CLK_IN: now also R11.1
- net VCXO_IN_T: no longer names the net of U3.3 (A0(A)/VC(B)/~{OEB}(C))
- net VCXO_IN_T: now also JP2.2 (C)
- new net: R2.1, R3.2, U2.4 (ADJ)
- new net: D5.2 (A), D6.2 (A), R2.2, U2.5 (OUT)
- new net: J5.2 (Pin_2), J5.4 (Pin_4), Q3.4 (S), U5.1 (S), U5.4 (EN), U5.6 (IN)
- new net: Q3.5 (G), U5.2 (G)
- new net: JP1.3 (B), JP2.1 (A), R11.2, R12.2, R13.1
- new net: Q3.2 (G), U1.2 (G)
- new net: JP1.2 (C), U3.6 ([~{OEB}(AB)]/CLKIN(C))
Other:
- note added: "+24V → +5V LDO"
- note added: "Ideal Diode"
- note added: "Si5351 Features Selectable Internal Capacitors External Load Capacitors Likely Unnecessary ...But Pads Are Available"
- note added: "Used If Powered From 3V3 With 5V Disabled"
- note removed: "Overvoltage Protection"
- note removed: "Si5351 Features Selectable Internal Capacitors External Load Capacitors Likely Unnecessary"
- moved on the sheet: C1, C10, C11, C12, C13, C14, C15, C16, C17, C18, C19, C2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

Commit message: Added solderpad jumpers
Parts:
- JP1: renamed from JP2; footprint (none) -> Jumper:SolderJumper-3_P2.0mm_Open_TrianglePad1.0x1.5mm
- JP2: renamed from JP1; footprint (none) -> Jumper:SolderJumper-3_P2.0mm_Open_TrianglePad1.0x1.5mm
- renumbered C38 to C1, C9 to C10, C10 to C11, C11 to C12, C12 to C13, C13 to C14, C14 to C15, C15 to C16, C16 to C17, C17 to C18, C18 to C19, C1 to C2, C19 to C20, C20 to C21, C21 to C22, C22 to C23, C23 to C24, C24 to C25, C25 to C26, C26 to C27, C27 to C28, C28 to C29, C2 to C3, C29 to C30, C30 to C31, C31 to C32, C32 to C33, C33 to C34, C34 to C35, C35 to C36, C36 to C37, C37 to C38, C3 to C4, C4 to C5, C5 to C6, C6 to C7, C7 to C8, C8 to C9, D4 to D1, D11 to D10, D6 to D4, D7 to D6, D8 to D7, D9 to D8, D10 to D9, J4 to J3, J5 to J4, J3 to J5, Q3 to Q1, R11 to R1, R8 to R10, R9 to R11, R10 to R12, R13 to R2, R12 to R3, R2 to R4, R3 to R5, R4 to R6, R5 to R7, R6 to R8, R7 to R9, U5 to U1, U1 to U2, U2 to U3, U3 to U4, U4 to U5

Commit message: PCB layout begins
Parts:
- S1: footprint Connector_PinHeader_1.00mm:PinHeader_1x01_P1.00mm_Horizontal -> libraries:Breadboard_400
Connections:
- net GND: now also J2.MP
Changed lines of the file:
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@@
 	)
 	(symbol
+		(lib_id "power:GND")
+		(at 24.13 119.38 0)
+		(unit 1)
+		(body_style 1)
+		(exclude_from_sim no)
+		(in_bom yes)
+		(on_board yes)
+		(in_pos_files yes)
+		(dnp no)
+		(fields_autoplaced yes)
+		(property "Reference" "#PWR064"
+			(at 24.13 125.73 0)
+			(hide yes)
+			(show_name no)
+			(do_not_autoplace no)
+			(effects
+				(font
+					(size 1.27 1.27)
+				)
+			)
+		)
+		(property "Value" "GND"
+			(at 24.13 122.5549 90)
+			(hide yes)
+			(show_name no)
+			(do_not_autoplace no)
+			(effects
+				(font
+					(size 1.27 1.27)
+				)
+				(justify right)
+			)
+		)
+		(property "Footprint" ""
+			(at 24.13 119.38 0)
+			(hide yes)
+			(show_name no)
+			(do_not_autoplace no)
+			(effects
+				(font
+					(size 1.27 1.27)
+				)
+			)
+		)
+		(property "Datasheet" ""
+			(at 24.13 119.38 0)
+			(hide yes)
+			(show_name no)
+			(do_not_autoplace no)
+			(effects
+				(font
+					(size 1.27 1.27)
+				)
+			)
+		)
+		(property "Description" ""
+			(at 24.13 119.38 0)
+			(show_name no)
+			(do_not_autoplace no)
+			(effects
+				(font
+					(size 1.27 1.27)
+				)
+			)
+		)
+		(pin "1"
+		)
+		(instances
+			(project "ClockGen_Si5351X_QFN16"
+				(path "/2b6c9482-e0ae-41e4-803d-260bc3a98f79"
+					(reference "#PWR064")
+					(unit 1)
+				)
+			)
+		)
+	)
+	(symbol
 		(lib_id "Device:C_Small")
 		(at 311.15 53.34 90)
@@
 		(pin "4"
 		)
+		(pin "MP"
+		)
 		(instances
 			(project "ClockGen_Si5351X_QFN16"
@@
 			)
 		)
-		(property "Footprint" "Connector_PinHeader_1.00mm:PinHeader_1x01_P1.00mm_Horizontal"
+		(property "Footprint" "libraries:Breadboard_400"
 			(at 300.99 243.84 0)
 			(hide yes)

Commit message: PCB Layout Progress
Parts:
- added J10, J11, J12, J13, J14: 2.54mm Stackable Socket, Connector_PinSocket_2.54mm:PinSocket_1x03_P2.54mm_Vertical, symbol Connector_Generic:Conn_01x03
- C17, C18, C19, C20, C21, C22, C23, C24, C25, C26, C27, C28, C29, C30, C31, C32, C33, C34: value 0402 -> 0402/0603; footprint libraries:Worthington_C_0402 -> libraries:Worthington_C_0402_0603
- SW1: footprint Button_Switch_THT:SW_Slide_SPDT_Angled_CK_OS102011MA1Q -> Button_Switch_THT:SW_Slide_SPDT_Straight_CK_OS102011MS2Q
Connections:
- net CLK0_BANDPASS: now also J10.1 (Pin_1), J10.2 (Pin_2), J10.3 (Pin_3)
- net CLK1_LOWPASS: now also J11.1 (Pin_1), J11.2 (Pin_2), J11.3 (Pin_3)
- net CLK2_BANDSTOP: now also J12.1 (Pin_1), J12.2 (Pin_2), J12.3 (Pin_3)
- net CLK3_HIGHPASS: now also J13.1 (Pin_1), J13.2 (Pin_2), J13.3 (Pin_3)
- net VCXO_IN/CLK_IN: now also J14.1 (Pin_1), J14.2 (Pin_2), J14.3 (Pin_3)
Other:
- moved on the sheet: D1, D10, D7, D8, D9

Commit message: PCB layout progress
Connections:
- net +3V0: now also RN1.4; no longer RN1.3
- net +5V_I2C_PULLUP: now also RN1.3; no longer RN1.4
- net I2C_SCL: now also RN1.7 (5); no longer RN1.6
- net I2C_SCL_5V: now also RN1.8; no longer RN1.5
- net I2C_SDA: now also RN1.5; no longer RN1.7 (5)
- net I2C_SDA_5V: now also RN1.6; no longer RN1.8
- net VCC: now also C2.1, J2.2 (Pin_2), Q1.6 (D), U2.3 (D), U3.1 (IN), U3.3 (EN); no longer J1.2 (Pin_2), Q1.1 (S), U2.1 (S), U2.4 (EN), U2.6 (IN)
- net +3V3: now reaches J4.2 (Pin_2), J4.4 (Pin_4), Q1.4 (S), U1.1 (S), U1.4 (EN), U1.6 (IN)
- new net: J1.2 (Pin_2), Q1.1 (S), U2.1 (S), U2.4 (EN), U2.6 (IN)
Other:
- moved on the sheet: RN1A, RN1B, RN1C, RN1D

Commit message: Most PCB layout done
Parts:
- C35, C36, C37, C38: footprint libraries:Worthington_C_0402 -> libraries:Worthington_C_0402_0603
- R2, R3: footprint libraries:Worthington_R_0201 -> libraries:Worthington_R_0402
Connections:
- net CLK0: now also C20.1; no longer C17.1, C22.1, L2.2
- net CLK3: now also C17.1, C22.1, L2.2; no longer C20.1
- net at C38.1: now also C34.1, L15.2, L16.2; no longer C33.2
- net CLK0_BANDPASS renamed CLK0_HIGHPASS
- net CLK3_HIGHPASS renamed CLK3_BANDPASS
- new net: C33.2, C35.1
Other:
- moved on the sheet: C17, C20, C22, C25, C27, C30, C31, C33, C34, L10, L12, L14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
