File: Modules/ClockGen_Si5351X_QFN16/ClockGen_Si5351X_QFN16.kicad_pcb (KiCad board)
At the start: 4 copper layers, 66.8 x 38.1 mm, 113 parts, among them J1 Screw Terminal, J10 2.54mm Stackable Socket, J11 2.54mm Stackable Socket, J12 2.54mm Stackable Socket, J13 2.54mm Stackable Socket, J14 2.54mm Stackable Socket, J2 JST SH, J3 SMA, J4 2.54 Pins, J5 2.54 Pins, J6 SMA, J7 SMA, J8 SMA, J9 SMA, Q1 GSFJ0300, Q2 GSFJ0300, SW1 SW_SPDT, U1 NCV68061, U2 NCV68061, U3 TPS7E8201, U4 SI5351B-B-GM1, U5 AP2127K-ADJ, U6 LM66200, Y1 25MHz

Commit message: RTL Module Schematic
Changed lines of the file:
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@@
-	)
-	(segment
-		(start 150.847219 115.090781)
-		(end 151.13 114.808)
-		(width 0.5)
-		(layer "F.Cu")
-		(net "/CLK1_LOWPASS")
 	)
 	(segment

Commit message: Fixed NCV68601 Footprint
Had the wrong pinout, glad I caught this!
Parts:
- C1, C10, C11, C12, C13, C16, C2, C3, C39, C4, C5: footprint libraries:Worthington_C_0402 -> libraries:Worthington_C_Narrow_0402
- C15, C6, C7, C8, C9: footprint libraries:Worthington_C_0201 -> libraries:Worthington_C_Narrow_0201
- C17, C18, C19, C20, C21, C22, C23, C24, C25, C26, C27, C28, C29, C30, C31, C32, C33, C34, C35, C36, C37, C38: footprint libraries:Worthington_C_0402_0603 -> libraries:Worthington_C_Narrow_0402_0603
- L1, L10, L11, L12, L13, L14, L15, L16, L2, L3, L4, L5, L6, L7, L8, L9: footprint libraries:Worthington_L_0603_RF -> libraries:Worthington_L_Narrow_0603_RF
- R1, R10, R11, R2, R3, R8, R9: footprint libraries:Worthington_R_0402 -> libraries:Worthington_R_Narrow_0402
- R12, R13, R14, R4, R5, R6, R7: footprint libraries:Worthington_R_0201 -> libraries:Worthington_R_Narrow_0201
- moved C1 0.14 mm to (136.7, 109.9)
- moved D1 0.10 mm to (148.9, 87.3)
- moved R14 0.07 mm to (146.2, 106.3)
- turned U2 to 90 degrees
Connections:
- U1 pad 2: Net-(Q1B-G) -> GND
- U1 pad 3: +5V_INT -> Net-(J5-Pin_2)
- U1 pad 4: Net-(J5-Pin_2) -> +5V_INT
- U1 pad 5: GND -> Net-(Q1B-G)
- U2 pad 2: Net-(Q1A-G) -> GND
- U2 pad 3: Net-(D12-K) -> /PWR_IN
- U2 pad 4: /PWR_IN -> Net-(D12-K)
- U2 pad 5: GND -> Net-(Q1A-G)
Routing:
- net GND: track 82.2 -> 144.6 mm, vias 167 -> 158
- net /PWR_IN: track 46.8 -> 99.2 mm, vias 2 -> 3
- net +5V_INT: track 68.0 -> 75.6 mm
- net Net-(J5-Pin_2): track 52.4 -> 58.0 mm
- net +3V3: track 88.1 -> 92.8 mm
- net Net-(Q1B-G): track 2.17 -> 6.28 mm
- net /I2C_SCL: track 13.4 -> 15.8 mm
- net Net-(Q1A-G): track 10.7 -> 12.1 mm
- net Net-(U6-ST): track 1.17 -> 2.61 mm
- net /I2C_SDA: track 19.2 -> 20.5 mm
- net Net-(U3-ADJ): track 9.13 -> 10.3 mm
- net /CLK3_BANDPASS: track 21.0 -> 22.1 mm
- net /CLK0_HIGHPASS: track 12.7 -> 13.7 mm
- net Net-(D6-K): track 3.45 -> 4.51 mm
- net /CLK1_LOWPASS: track 12.9 -> 13.9 mm
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- added copper zone on B.Cu, net /PWR_IN
Other:
- board text removed: "L"

Commit message: Added input power snubber
Just in case :P
Parts:
- added C40: 47u, libraries:Worthington_C_0805, F.Cu at (137.4, 102.2)
- added R15: 1R, Resistor_SMD:R_0805_2012Metric, F.Cu at (134.3, 102.2)
Routing:
- net /PWR_IN: track 99.2 -> 102.9 mm
- net Net-(C40-Pad2): track 0.00 -> 1.21 mm
